File: Cheshire50.kicad_pcb (KiCad board)
At the start: 2 copper layers, 318.2 x 103.5 mm, 135 parts, among them J1 JST_DB, J2 JST_PCB, SW1 MX_SW_HS, SW10 MX_SW_HS, SW11 MX_SW_HS, SW12 MX_SW_HS, SW13 MX_SW_HS, SW14 MX_SW_HS, SW15 MX_SW_HS, SW16 MX_SW_HS, SW17 MX_SW_HS, SW18 MX_SW_HS, SW19 MX_SW_HS, SW2 MX_SW_HS, SW20 MX_SW_HS, SW21 MX_SW_HS, SW22 MX_SW_HS, SW23 MX_SW_HS, SW24 MX_SW_HS, SW25 MX_SW_HS, SW26 MX_SW_HS, SW27 MX_SW_HS, SW28 MX_SW_HS, SW29 MX_SW_HS, SW3 MX_SW_HS, SW30 MX_SW_HS, SW31 MX_SW_HS, SW32 MX_SW_HS, SW33 MX_SW_HS, SW34 MX_SW_HS, SW35 MX_SW_HS, SW36 MX_SW_HS, SW37 MX_SW_HS, SW38 MX_SW_HS, SW39 MX_SW_HS, SW4 MX_SW_HS, SW40 MX_SW_HS, SW41 MX_SW_HS, SW42 MX_SW_HS, SW43 MX_SW_HS, SW44 MX_SW_HS, SW45 MX_SW_HS, SW46 MX_SW_HS, SW47 MX_SW_HS, SW48 MX_SW_HS, SW49 MX_SW_HS, SW5 MX_SW_HS, SW50 MX_SW_HS, SW51 MX_SW_HS, SW52 MX_SW_HS, SW53 MX_SW_HS, SW54 MX_SW_HS, SW55 MX_SW_HS, SW56 SW_Push, SW6 MX_SW_HS, SW7 MX_SW_HS, SW8 MX_SW_HS, SW9 MX_SW_HS, U1 ATMEGA32U4-AU, U2 PRTR5V0U2X, Y1 16MHz

Commit message: new routing and logo
Parts:
- removed the SW13 at (289.4, 25.7)
- added REF** (x2): Cheshire50Logo, Cheshire:Cheshire50Logo, F.Cu at (147.8, 22.2)
- D1, D10, D11, D12, D13, D14, D15, D16, D17, D18, D19, D2, D20, D21, D22, D23, D24, D25, D26, D27, D28, D29, D3, D30, D31, D32, D33, D34, D35, D36, D37, D38, D39, D4, D40, D41, D42, D43, D44, D45, D46, D47, D48, D49, D5, D50, D51, D52, D53, D54, D55, D6, D7, D8, D9: footprint Keebio-Parts:Diode-Hybrid-Back -> Keebio-Parts:Diode-dual
- moved C1 4.59 mm to (141.0, 44.5)
- moved R2 4.43 mm to (138.4, 23.2)
- moved R4 2.07 mm to (142.9, 24.8)
- moved R3 1.11 mm to (135.9, 23.1)
- moved Y1 0.84 mm to (152.4, 23.5)
- moved C6 0.68 mm to (156.2, 22.2)
- moved R1 0.68 mm to (154.7, 42.0)
- moved U1 0.68 mm to (147.3, 35.4)
- moved D23 0.51 mm to (189.9, 60.3)
- moved D26 0.46 mm to (248.6, 53.3)
- moved D19 0.39 mm to (91.8, 57.1)
- moved D13 0.33 mm to (278.3, 14.0)
- moved D24 0.28 mm to (208.5, 57.1)
- moved D18 0.19 mm to (73.0, 54.0)
- moved D12 0.17 mm to (259.6, 33.7)
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- renumbered SW56 to RESET1
Connections:
- RES1 pad S1: COL 14 -> ROW 0
- RES1 pad S2: ROW 0 -> COL 13
- U1 pad 12: COL 7 -> unconnected-(U1-PB7-Pad12)
- U1 pad 26: unconnected-(U1-PD6-Pad26) -> COL 9
- U1 pad 27: unconnected-(U1-PD7-Pad27) -> COL 8
- U1 pad 28: COL 4 -> COL 7
- U1 pad 29: COL 5 -> COL 6
- U1 pad 30: COL 6 -> unconnected-(U1-PB6-Pad30)
Routing:
- net ROW 3: track 0.00 -> 353.9 mm, vias 0 -> 2
- net ROW 0: track 0.00 -> 340.1 mm, vias 0 -> 3
- net ROW 2: track 0.00 -> 325.7 mm, vias 0 -> 2
- net ROW 1: track 0.00 -> 297.5 mm, vias 0 -> 2
- net GND: track 153.2 -> 348.7 mm, vias 5 -> 8
- net COL 0: track 0.00 -> 190.9 mm
- net RES1 A: track 0.00 -> 182.6 mm
- net RES1 B: track 0.00 -> 173.5 mm
- net COL 1: track 0.00 -> 172.3 mm
- net COL 2: track 0.00 -> 152.5 mm
- net COL 3: track 0.00 -> 150.5 mm
- net COL 9: track 0.00 -> 139.8 mm
- net COL 8: track 0.00 -> 126.3 mm
- net COL 7: track 0.00 -> 94.4 mm
- net COL 13: track 146.1 -> 230.0 mm
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Other:
- board text added: "CHESHIRE50"

Commit message: rewire to reduce pcb width ... by 5mm
Parts:
- removed REF** (x2): Cheshire50Logo, Cheshire:Cheshire50Logo
- moved R2 25.0 mm to (144.8, 47.3)
- moved R1 24.1 mm to (156.2, 66.0), turned to 180 degrees
- moved R3 23.2 mm to (141.0, 45.7)
- moved Y1 22.2 mm to (152.4, 45.7)
- moved U1 21.9 mm to (149.9, 57.1)
- moved D15 21.7 mm to (301.0, 35.6)
- moved C6 18.8 mm to (152.4, 40.6), turned to 180 degrees
- moved C7 17.4 mm to (147.3, 41.9), turned to 90 degrees
- moved RESET1 17.0 mm to (147.3, 39.4)
- moved J2 15.0 mm to (146.6, 31.6)
- moved R4 14.7 mm to (141.0, 39.4), turned to 180 degrees
- moved D13 6.35 mm to (278.3, 20.3)
- moved C1 6.35 mm to (141.0, 50.8)
- moved J1 5.88 mm to (318.0, 26.8)
- moved R6 5.88 mm to (325.0, 36.8)
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Routing:
- net 5V: track 63.5 -> 97.8 mm
- net GND: track 348.7 -> 376.6 mm, vias 8 -> 7
- net ROW 2: track 325.7 -> 303.6 mm
- net ROW 3: track 353.9 -> 332.2 mm
- net RES1 B: track 173.5 -> 189.9 mm, vias 0 -> 2
- net ROW 0: track 340.1 -> 355.1 mm, vias 3 -> 4
- net COL 6: track 75.4 -> 90.0 mm
- net Net-(U1-~{RESET}): track 9.42 -> 21.3 mm
- net COL 3: track 150.5 -> 138.7 mm, vias 0 -> 1
- net RES1 A: track 182.6 -> 194.3 mm, vias 0 -> 2
- net COL 12: track 208.1 -> 196.4 mm, vias 0 -> 1
- net Net-(D15-A): track 17.3 -> 6.10 mm
- net D-: track 14.1 -> 23.9 mm
- net COL 9: track 139.8 -> 131.6 mm, vias 0 -> 1
- net Net-(D13-A): track 17.7 -> 10.7 mm
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Other:
- board size 318.2 x 103.5 mm -> 313.6 x 96.7 mm
- board text removed: "CHESHIRE50"

Commit message: rerouting, moved daughterboard to bottom to save space
Parts:
- moved USB1 107.3 mm to (272.1, 115.5), turned to 0 degrees
- moved C5 100.6 mm to (282.1, 107.9), turned to 90 degrees
- moved F1 99.1 mm to (278.7, 107.9), turned to 90 degrees
- moved U2 95.2 mm to (265.1, 107.9), turned to 0 degrees
- moved R6 95.0 mm to (262.1, 108.0), turned to 90 degrees
- moved C3 94.4 mm to (282.1, 103.2), turned to 90 degrees
- moved C2 93.3 mm to (279.9, 103.2), turned to 90 degrees
- moved C4 89.4 mm to (264.4, 103.9), turned to 90 degrees
- moved R5 89.2 mm to (262.1, 103.9), turned to -90 degrees
- moved J1 87.3 mm to (272.1, 101.0), turned to 0 degrees
- moved ? 80.1 mm to (275.1, 94.8), turned to 0 degrees
- moved ? 77.8 mm to (268.7, 94.8), turned to 0 degrees
Routing:
- net Net-(U1-~{RESET}): track 21.3 -> 30.1 mm
- net GND: track 376.6 -> 370.2 mm, vias 7 -> 5
- net COL 10: track 141.1 -> 137.3 mm
- net 5V: track 97.8 -> 99.2 mm
- net COL 2: track 154.8 -> 153.5 mm
- net COL 6: track 90.0 -> 90.9 mm
- net COL 0: track 195.5 -> 196.1 mm
Other:
- board size 313.6 x 96.7 mm -> 292.1 x 101.1 mm
